File: assets/pcb/verbum-horolgium.kicad_pcb (KiCad board)
At the start: 2 copper layers, 100 x 100 mm, 33 parts, among them J1 GND, J2 +5V, J3 LED_DATA, J4 TOUCH, J5 POWER (6-32V), J6 POWER (6-32V), U1 AP63205WU-7

Commit message: chore: added text to front silkscreen
Parts:
- moved TP4 34.1 mm to (131.2, 149.2)
Other:
- board text added: "+5V"
- board text added: "6-32V"
- board text added: "GND"
- board text added: "LEFT"
- board text added: "RIGHT"
- board text added: "TOP"
Changed lines of the file:
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@@
 			)
 		)
-		(attr smd dnp)
+		(attr smd)
 		(duplicate_pad_numbers_are_jumpers no)
 		(fp_line
@@
 	(footprint "Connector_PinHeader_1.00mm:PinHeader_1x01_P1.00mm_Vertical"
 		(layer "F.Cu")
-		(at 106.194 125.993)
+		(at 131.191 149.225)
 		(descr "Through hole straight pin header, 1x01, 1.00mm pitch, single row")
 		(tags "Through hole pin header THT 1x01 1.00mm single row")
@@
 			)
 		)
-		(attr through_hole)
+		(attr through_hole exclude_from_bom)
 		(duplicate_pad_numbers_are_jumpers no)
 		(fp_line
@@
 			)
 		)
-		(attr through_hole)
+		(attr through_hole exclude_from_bom)
 		(duplicate_pad_numbers_are_jumpers no)
 		(fp_line
@@
 			)
 		)
-		(attr through_hole)
+		(attr through_hole exclude_from_bom)
 		(duplicate_pad_numbers_are_jumpers no)
 		(fp_line
@@
 			)
 		)
-		(attr through_hole)
+		(attr through_hole exclude_from_bom)
 		(duplicate_pad_numbers_are_jumpers no)
 		(fp_line
@@
 		(layer "Edge.Cuts")
 	)
+	(gr_text "GND"
+		(at 186.055 136 0)
+		(layer "F.SilkS")
+		(effects
+			(font
+				(size 1 1)
+				(thickness 0.15)
+			)
+			(justify left)
+		)
+	)
+	(gr_text "6-32V"
+		(at 186.055 141 0)
+		(layer "F.SilkS")
+		(effects
+			(font
+				(size 1 1)
+				(thickness 0.15)
+			)
+			(justify left)
+		)
+	)
+	(gr_text "GND"
+		(at 186.055 146 0)
+		(layer "F.SilkS")
+		(effects
+			(font
+				(size 1 1)
+				(thickness 0.15)
+			)
+			(justify left)
+		)
+	)
+	(gr_text "6-32V"
+		(at 186.055 151 0)
+		(layer "F.SilkS")
+		(effects
+			(font
+				(size 1 1)
+				(thickness 0.15)
+			)
+			(justify left)
+		)
+	)
+	(gr_text "+5V"
+		(at 186.195286 122.809 0)
+		(layer "F.SilkS")
+		(effects
+			(font
+				(size 1.5 1.5)
+				(thickness 0.15)
+			)
+			(justify left)
+		)
+	)
+	(gr_text "GND"
+		(at 108.444 122.809 0)
+		(layer "F.SilkS")
+		(effects
+			(font
+				(size 1.5 1.5)
+				(thickness 0.15)
+			)
+		)
+	)
 	(gr_text "${COMPANY}"
 		(at 100.838 135.509 0)
 		(layer "F.SilkS")
 		(effects
+			(font
+				(size 1.5 1.5)
+				(thickness 0.1875)
+			)
+			(justify left)
+		)
+	)
+	(gr_text "LEFT"
+		(at 118.502857 141 0)
+		(layer "F.SilkS")
+		(effects
+			(font
+				(size 1.5 1.5)
+				(thickness 0.1875)
+			)
+			(justify left)
+		)
+	)
+	(gr_text "RIGHT"
+		(at 118.502857 146 0)
+		(layer "F.SilkS")
+		(effects
+			(font
+				(size 1.5 1.5)
+				(thickness 0.1875)
+			)
+			(justify left)
+		)
+	)
+	(gr_text "TOP"
+		(at 118.502857 151 0)
+		(layer "F.SilkS")
+		(effects
