File: assets/pcb/verbum-horolgium.kicad_sch (KiCad schematic)
At the start: 1 part

Commit message: chore: basic schematic complete
Parts:
- added A2: CAP1188, verbum-horologium_footprints:CAP1188-breakout, symbol verbum-horologium_symbols:CAP1188-breakout
- added A3: DS3231, verbum-horologium_footprints:DS3231-breakout, symbol verbum-horologium_symbols:DS3231-breakout
- added C1: 10u, Capacitor_SMD:C_1210_3225Metric, symbol Device:C
- added C2, C4: 22u, Capacitor_SMD:C_1206_3216Metric, symbol Device:C
- added C3, C6, C7: 1000u, Capacitor_SMD:CP_Elec_10x10, symbol Device:C_Polarized
- added C5: 100n, Capacitor_SMD:C_0805_2012Metric, symbol Device:C
- added D1: POWER, LED_SMD:LED_1206_3216Metric, symbol Device:LED
- added D2: ACTIVITY, LED_SMD:LED_1206_3216Metric, symbol Device:LED
- added D3: V1P6-M3/H, Diode_SMD:D_MicroSMP_LargeCathode, symbol Device:D_Schottky
- added F1: 2.5A, Fuse:Fuse_0603_1608Metric, symbol Device:Fuse
- added J1: GND, verbum-horologium_footprints:SolderWire-1.5sqmm_1x13_P6mm_D1.7mm_OD3mm_Relief, symbol Connector_Generic:Conn_01x13
- added J2: +5V, verbum-horologium_footprints:SolderWire-1.5sqmm_1x13_P6mm_D1.7mm_OD3mm_Relief, symbol Connector_Generic:Conn_01x13
- added J3: LED_DATA, Connector_Wire:SolderWire-1.5sqmm_1x01_D1.7mm_OD3mm_Relief, symbol Connector_Generic:Conn_01x01
- added J4: TOUCH, Connector_Wire:SolderWire-1.5sqmm_1x03_P6mm_D1.7mm_OD3mm_Relief, symbol Connector_Generic:Conn_01x03
- added J5, J6: POWER (6-32V), Connector_Wire:SolderWire-1.5sqmm_1x02_P7.8mm_D1.7mm_OD3.9mm_Relief, symbol Connector_Generic:Conn_01x02
- added JP2: VBUS, Jumper:SolderJumper-2_P1.3mm_Open_TrianglePad1.0x1.5mm, symbol Jumper:SolderJumper_2_Open
- added L1: 10u, verbum-horologium_footprints:L_Wurth_WE-TPC-1038, symbol Device:L
- added R1: R, Resistor_THT:R_Axial_DIN0207_L6.3mm_D2.5mm_P7.62mm_Horizontal, symbol Device:R
- added R2: 18-44k, Connector_Wire:SolderWire-1.5sqmm_1x02_P6mm_D1.7mm_OD3mm_Relief, symbol Device:R_Photo
- added R3, R4: 180, Resistor_SMD:R_0603_1608Metric, symbol Device:R
- added R5: 20k, Resistor_THT:R_Axial_DIN0207_L6.3mm_D2.5mm_P7.62mm_Horizontal, symbol Device:R
- added U1: AP63205WU-7, SOIC_05WU-7_DIO, symbol verbum-horologium_symbols:AP63205WU-7
- A1: PN (none) -> SC0915
Connections:
- net FRONT_SENSOR: now also R2.2, R5.2
- net LED_DATA: now reaches A1.10 (GPIO7)
- net LED_DATA: now also R1.1
- net GND: now reaches A1.13 (GND), A1.18 (GND), A1.23 (GND), A1.28 (GND), A1.3 (GND), A1.38 (GND), A1.8 (GND)
- net GND: now also A2.4 (GND), A3.2 (GND), C1.2, C2.2, C3.2, C4.2, C6.2, C7.2, D1.1 (K), D2.1 (K), J1.1 (Pin_1), J1.10 (Pin_10), J1.11 (Pin_11), J1.12 (Pin_12), J1.13 (Pin_13), J1.2 (Pin_2), J1.3 (Pin_3), J1.4 (Pin_4), J1.5 (Pin_5), J1.6 (Pin_6), J1.7 (Pin_7), J1.8 (Pin_8), J1.9 (Pin_9), J5.2 (Pin_2), J6.2 (Pin_2), R5.1, U1.4 (GND)
- net ACTIVITY: now reaches A1.14 (GPIO10)
- net ACTIVITY: now also R4.1
- net at A1.39 (VSYS): now also D3.1 (K)
- net at A1.40 (VBUS): now also JP2.1 (A)
- net SDA: now reaches A1.6 (GPIO4)
- net SDA: now also A2.1 (SDA), A3.4 (SDA)
- net SCL: now reaches A1.7 (GPIO5)
- net SCL: now also A2.2 (SCK), A3.3 (SCL)
- new net: D1.2 (A), R3.2
- new net: A2.20 (C3), J4.3 (Pin_3)
- new net: A2.21 (C2), J4.2 (Pin_2)
- new net: A2.22 (C1), J4.1 (Pin_1)
- new net: D2.2 (A), R4.2
- new net: C5.1, U1.6 (BST)
- new net: C5.2, L1.1, U1.5 (SW)
- new net: C1.1, F1.2, U1.2 (EN), U1.3 (VIN)
- new net: J3.1 (Pin_1), R1.2
- new net +5V: A2.3 (VIN), A3.1 (VIN), C2.1, C3.1, C4.1, C6.1, C7.1, D3.2 (A), J2.1 (Pin_1), J2.10 (Pin_10), J2.11 (Pin_11), J2.12 (Pin_12), J2.13 (Pin_13), J2.2 (Pin_2), J2.3 (Pin_3), J2.4 (Pin_4), J2.5 (Pin_5), J2.6 (Pin_6), J2.7 (Pin_7), J2.8 (Pin_8), J2.9 (Pin_9), JP2.2 (B), L1.2, R2.1, R3.1, U1.1 (FB)
- new net VDD: F1.1, J5.1 (Pin_1), J6.1 (Pin_1)
- no-connect marks 0 -> 47
Other:
- note added: "18AWG"
- moved on the sheet: A1

Commit message: chore: pcb layout complete
Parts:
- added TP1, TP2, TP3, TP4: (no value), Connector_PinHeader_1.00mm:PinHeader_1x01_P1.00mm_Vertical, symbol Connector:TestPoint
- J1, J2: footprint verbum-horologium_footprints:SolderWire-1.5sqmm_1x13_P6mm_D1.7mm_OD3mm_Relief -> verbum-horologium_footprints:SolderWire-1.5sqmm_1x13_P5mm_D1.7mm_OD3mm_Relief
- J3: footprint Connector_Wire:SolderWire-1.5sqmm_1x01_D1.7mm_OD3mm_Relief -> verbum-horologium_footprints:SolderWire-1.5sqmm_1x1_P5mm_D1.7mm_OD3mm_Relief
- J4: footprint Connector_Wire:SolderWire-1.5sqmm_1x03_P6mm_D1.7mm_OD3mm_Relief -> verbum-horologium_footprints:SolderWire-1.5sqmm_1x3_P5mm_D1.7mm_OD3mm_Relief
- J5, J6: footprint Connector_Wire:SolderWire-1.5sqmm_1x02_P7.8mm_D1.7mm_OD3.9mm_Relief -> verbum-horologium_footprints:SolderWire-1.5sqmm_1x2_P5mm_D1.7mm_OD3mm_Relief
- R2: footprint Connector_Wire:SolderWire-1.5sqmm_1x02_P6mm_D1.7mm_OD3mm_Relief -> verbum-horologium_footprints:SolderWire-1.5sqmm_1x2_P5mm_D1.7mm_OD3mm_Relief
Connections:
- net +5V: now also TP1.1
- net FRONT_SENSOR: now also TP3.1
- net GND: now also TP4.1
- net at A2.20 (C3): now also J4.1 (Pin_1); no longer J4.3 (Pin_3)
- net at A2.22 (C1): now also J4.3 (Pin_3); no longer J4.1 (Pin_1)
- net at C1.1, F1.2, U1.2 (EN)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: now also TP2.1
Other:
- moved on the sheet: F1

Commit message: chore: added text to front silkscreen
Parts:
- U1: footprint SOIC_05WU-7_DIO -> verbum-horologium_footprints:SOIC_05WU-7_DIO
Changed lines of the file:
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@@
 			)
 		)
-		(property "Footprint" "SOIC_05WU-7_DIO"
+		(property "Footprint" "verbum-horologium_footprints:SOIC_05WU-7_DIO"
 			(at 123.19 63.5 0)
 			(hide yes)

Commit message: fix: added mounting holes
Parts:
- added H1, H2, H3, H4: MountingHole, MountingHole:MountingHole_3.2mm_M3, symbol Mechanical:MountingHole
